File: KubkuinoDNO_GY-906/Board_KiCAD_GY-906/Board.sch (KiCad schematic (older format))
At the start: 33 parts, among them J1 Piezo, J2 AC/DC In (12V), J3 Prog, J4 Czujnik, J6 LCD, J7 Button, J8 Bluetooth, Q1 S8050, SW1 Reset, U1 LM7805_TO220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

Commit message: Fixed SMD board
Parts:
- removed U2: ATMEGA328P-PU, Housings_QFP:TQFP-32_7x7mm_Pitch0.8mm, symbol ATMEGA328P-PU
- added RJ2: 0, Resistors_SMD:R_1206, symbol R
- added U2: ATMEGA328P-AU, Housings_QFP:TQFP-32_7x7mm_Pitch0.8mm, symbol ATMEGA328P-AU
- RJ1: footprint (none) -> Resistors_SMD:R_1206
- SW1: footprint Buttons_Switches_SMD:SW_SPST_B3SL-1002P -> Buttons_Switches_THT:SW_PUSH_6mm_h5mm
- Y1: footprint Crystals:Crystal_SMD_HC49-SD -> Crystals:Crystal_SMD_HC49-SD_HandSoldering
Connections:
- wire segments 40 -> 43
Other:
- moved on the sheet: C5, C6, D7, D8, D9, J1, J3, J4, J6, J7, J8, Q1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
