File: KubkuinoDNO_GY-906/Board_KiCAD_GY-906/Board.sch (KiCad schematic (older format))
At the start: 34 parts, among them J1 Piezo, J2 AC/DC In (12V), J3 Prog, J4 Czujnik, J6 LCD, J7 Button, J8 Bluetooth, Q1 S8050, SW1 Reset, U1 LM7805_TO220, U2 ATMEGA328P-AU, Y1 Crystal

Commit message: Minor optimization
Board GY906:
Removed ICSP header and replaced with pads
Moved power input to the edge
Added fuse after LM7805

GY906 sketch:
Alarm has got new launch method (removed booleans)
Removed unused headers
Selected one tone frequency for buzzer
Some other things
Parts:
- removed J3: Prog, symbol CONN_02X03
- removed R5: 1k, Resistors_SMD:R_1206, symbol R
- removed RJ1, RJ2: 0, Resistors_SMD:R_1206, symbol R
- removed SW1: Reset, Buttons_Switches_THT:SW_PUSH_6mm_h5mm, symbol SW_Push
- added F1: 500mA 6V, SMD_Packages:SMD-1206_Pol, symbol Polyfuse
- added J2, J4: Conn_01x03, Socket_Strips:Socket_Strip_Straight_1x03_Pitch2.54mm, symbol Conn_01x03
- J6: renamed from J2; footprint Pin_Headers:Pin_Header_Straight_1x02_Pitch2.54mm_SMD_Pin1Left -> Socket_Strips:Socket_Strip_Angled_1x02_Pitch2.54mm
- renumbered D7 to D1, D8 to D2, D9 to D3, D1 to D4, D2 to D5, D3 to D6, D4 to D7, J4 to J3, J6 to J5, J8 to J7, J7 to J8, R6 to R5, R7 to R6, U2 to U1, U1 to U2
Connections:
- net 5V: now also F1.1, J4.1 (Pin_1); no longer C3.1, C4.1, U2.3 (VO)
- net GND: now also J4.3 (Pin_3)
- net Reset: now also J2.3 (Pin_3)
- net at D4.2 (A), D6.1 (K): now also J6.2 (P2); no longer J6.1 (P1)
- net at D5.2 (A), D7.1 (K): now also J6.1 (P1); no longer J6.2 (P2)
- net at U1.15 ((PCINT3/OC2A/MOSI)PB3): now also J4.2 (Pin_2)
- net at U1.16 ((PCINT4/MISO)PB4): now also J2.1 (Pin_1)
- net at U1.17 ((PCINT5/SCK)PB5): now also J2.2 (Pin_2)
- new net: C3.1, C4.1, F1.2, U2.3 (VO)
Other:
- moved on the sheet: D4, D5, D6, D7, J6, J8, R4

Commit message: Updates
Parts:
- removed J3: Czujnik, Pin_Headers:Pin_Header_Straight_1x04_Pitch2.54mm_SMD_Pin1Left, symbol CONN_01X04
- removed J5: LCD, Pin_Headers:Pin_Header_Straight_1x04_Pitch2.54mm_SMD_Pin1Left, symbol CONN_01X04
- added J3: I2C, Socket_Strips:Socket_Strip_Straight_2x04_Pitch2.54mm_SMD, symbol Conn_02x04_Odd_Even
Connections:
- net 5V: now also J3.7 (Pin_7), J3.8 (Pin_8)
- net GND: now also J3.5 (Pin_5), J3.6 (Pin_6)
- net SCL: now also J3.3 (Pin_3), J3.4 (Pin_4)
- net SDA: now also J3.1 (Pin_1), J3.2 (Pin_2)
- net at D4.2 (A), D6.1 (K): now also J6.1 (P1); no longer J6.2 (P2)
- net at D5.2 (A), D7.1 (K): now also J6.2 (P2); no longer J6.1 (P1)
Changed lines of the file:
@@
-EESchema Schematic File Version 2
+EESchema Schematic File Version 3
 LIBS:power
 LIBS:device
@@
 LIBS:ftdi
 LIBS:gennum
+LIBS:graphic
 LIBS:graphic_symbols
 LIBS:hc11
@@
 F 3 "" H 2450 5350 50  0001 C CNN
 	1    2450 5350
-	-1   0    0    1
+	-1   0    0    -1
 $EndComp
 Text GLabel 5450 5250 2    60   Input ~ 0
@@
 Bkey
 $Comp
-L CONN_01X04 J3
-U 1 1 597553D9
-P 5750 3000
-F 0 "J3" H 5750 3250 50  0000 C CNN
-F 1 "Czujnik" V 5850 3000 50  0000 C CNN
-F 2 "Pin_Headers:Pin_Header_Straight_1x04_Pitch2.54mm_SMD_Pin1Left" H 5750 3000 50  0001 C CNN
-F 3 "" H 5750 3000 50  0001 C CNN
-	1    5750 3000
-	1    0    0    -1
-$EndComp
-$Comp
-L CONN_01X04 J5
-U 1 1 597555A0
-P 6150 3000
-F 0 "J5" H 6150 3250 50  0000 C CNN
-F 1 "LCD" V 6250 3000 50  0000 C CNN
-F 2 "Pin_Headers:Pin_Header_Straight_1x04_Pitch2.54mm_SMD_Pin1Left" H 6150 3000 50  0001 C CNN
-F 3 "" H 6150 3000 50  0001 C CNN
-	1    6150 3000
-	1    0    0    -1
-$EndComp
-$Comp
 L GND #PWR06
 U 1 1 5975584B
-P 5550 3050
-F 0 "#PWR06" H 5550 2800 50  0001 C CNN
-F 1 "GND" H 5550 2900 50  0000 C CNN
-F 2 "" H 5550 3050 50  0001 C CNN
-F 3 "" H 5550 3050 50  0001 C CNN
-	1    5550 3050
-	0    1    1    0
-$EndComp
-Text GLabel 5550 3150 0    60   Input ~ 0
+P 5700 3050
+F 0 "#PWR06" H 5700 2800 50  0001 C CNN
+F 1 "GND" H 5700 2900 50  0000 C CNN
+F 2 "" H 5700 3050 50  0001 C CNN
+F 3 "" H 5700 3050 50  0001 C CNN
+	1    5700 3050
+	1    0    0    -1
+$EndComp
+Text GLabel 5950 3150 0    60   Input ~ 0
 5V
 Text GLabel 5300 2200 0    60   Input ~ 0
@@
 Text GLabel 4700 1600 2    60   Input ~ 0
 1W
-Text GLabel 6300 2850 2    60   Input ~ 0
+Text GLabel 6450 2850 2    60   Input ~ 0
 SDA
-Text GLabel 6300 2950 2    60   Input ~ 0
+Text GLabel 6450 2950 2    60   Input ~ 0
 SCL
 Text GLabel 4700 3600 2    60   Input ~ 0
@@
 	7550 2950 7550 3150
 Wire Wire Line
-	4700 2850 6300 2850
-Connection ~ 5550 2850
-Wire Wire Line
-	4700 2950 6300 2950
-Wire Wire Line
-	5550 3050 5950 3050
-Wire Wire Line
-	5950 3150 5550 3150
-Connection ~ 5550 2950
-Connection ~ 5950 2850
-Connection ~ 5950 2950
-Wire Wire Line
 	3900 5550 5050 5550
 Connection ~ 4100 5550
@@
 $EndComp
 Connection ~ 5050 5250
+Text GLabel 5950 2850 0    60   Input ~ 0
+SDA
+Text GLabel 5950 2950 0    60   Input ~ 0
+SCL
+Text GLabel 6450 3150 2    60   Input ~ 0
+5V
+Wire Wire Line
+	5700 3050 5950 3050
+$Comp
+L GND #PWR012
+U 1 1 59F4A174
+P 6700 3050
+F 0 "#PWR012" H 6700 2800 50  0001 C CNN
+F 1 "GND" H 6700 2900 50  0000 C CNN
+F 2 "" H 6700 3050 50  0001 C CNN
+F 3 "" H 6700 3050 50  0001 C CNN
+	1    6700 3050
+	1    0    0    -1
+$EndComp
+Wire Wire Line
+	6450 3050 6700 3050
+Text GLabel 5250 2950 2    60   Input ~ 0
+SDA
+Text GLabel 5250 3050 2    60   Input ~ 0
+SCL
+Wire Wire Line
+	4700 2850 4800 2850
+Wire Wire Line
+	4800 2850 4800 2900
+Wire Wire Line
+	4800 2900 5200 2900
+Wire Wire Line
+	5200 2900 5200 2950
+Wire Wire Line
+	5200 2950 5250 2950
+Wire Wire Line
+	4700 2950 5150 2950
+Wire Wire Line
+	5150 2950 5150 3050
+Wire Wire Line
+	5150 3050 5250 3050
+$Comp
+L Conn_02x04_Odd_Even J3
+U 1 1 59F4A6D7
+P 6150 2950
+F 0 "J3" H 6200 3267 50  0000 C CNN
+F 1 "I2C" H 6200 3176 50  0000 C CNN
+F 2 "Socket_Strips:Socket_Strip_Straight_2x04_Pitch2.54mm_SMD" H 6150 2950 50  0001 C CNN
+F 3 "" H 6150 2950 50  0001 C CNN
+	1    6150 2950
+	1    0    0    -1
+$EndComp
 $EndSCHEMATC
