File: KubkuinoDNO_GY-906/Board_KiCAD_GY-906/_saved_Board.sch (KiCad schematic (older format))
At the start: 34 parts, among them J1 Piezo, J2 AC/DC In (12V), J3 Prog, J4 Czujnik, J6 LCD, J7 Button, J8 Bluetooth, Q1 S8050, SW1 Reset, U1 LM7805_TO220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

Commit message: Finished PCB
Parts:
- J3: footprint (none) -> Pin_Headers:Pin_Header_Straight_2x03_Pitch2.54mm
Changed lines of the file:
@@
 F 0 "J3" H 6100 2150 50  0000 C CNN
 F 1 "Prog" H 6100 1750 50  0000 C CNN
-F 2 "" H 6100 750 50  0001 C CNN
+F 2 "Pin_Headers:Pin_Header_Straight_2x03_Pitch2.54mm" H 6100 750 50  0001 C CNN
 F 3 "" H 6100 750 50  0001 C CNN
 	1    6100 1950
